File: PCB/splitkeybaord.kicad_sch (KiCad schematic)
At the start: 0 parts

Commit message: minor update
Changed lines of the file:
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@@
 	(paper "A4")
 	(sheet
-		(at 20.32 107.95)
-		(size 99.06 73.66)
+		(at 23.495 19.05)
+		(size 162.56 59.69)
+		(exclude_from_sim no)
+		(in_bom yes)
+		(on_board yes)
+		(dnp no)
+		(fields_autoplaced yes)
+		(stroke
+			(width 0.1524)
+			(type solid)
+		)
+		(fill
+			(color 0 0 0 0)
+		)
+		(property "Sheetname" "left"
+			(at 23.495 18.3384 0)
+			(show_name no)
+			(do_not_autoplace no)
+			(effects
+				(font
+					(size 1.27 1.27)
+				)
+				(justify left bottom)
+			)
+		)
+		(property "Sheetfile" "keyboard.kicad_sch"
+			(at 23.495 79.3246 0)
+			(show_name no)
+			(do_not_autoplace no)
+			(effects
+				(font
+					(size 1.27 1.27)
+				)
+				(justify left top)
+			)
+		)
+		(instances
+			(project "splitkeybaord (3)"
+				(path "/667832f1-ce12-4971-b6ce-e9db115b7c92"
+					(page "2")
+				)
+			)
+		)
+	)
+	(sheet
+		(at 24.13 99.695)
+		(size 165.1 62.23)
 		(exclude_from_sim no)
 		(in_bom yes)
@@
 		)
 		(property "Sheetname" "right"
-			(at 20.32 107.2384 0)
+			(at 24.13 98.9834 0)
 			(show_name no)
 			(do_not_autoplace no)
@@
 		)
 		(property "Sheetfile" "keyboard.kicad_sch"
-			(at 20.32 182.1946 0)
+			(at 24.13 162.5096 0)
 			(show_name no)
 			(do_not_autoplace no)
@@
 		)
 		(instances
-			(project "split keyboard"
-				(path "/e1af24d2-b379-41bc-99d4-76686fb1dd1a"
+			(project "splitkeybaord (3)"
+				(path "/667832f1-ce12-4971-b6ce-e9db115b7c92"
 					(page "3")
 				)
 			)
-		)
-	)
-	(sheet
-		(at 22.86 25.4)
-		(size 97.79 67.31)
-		(exclude_from_sim no)
-		(in_bom yes)
-		(on_board yes)
-		(dnp no)
-		(fields_autoplaced yes)
-		(stroke
-			(width 0.1524)
-			(type solid)
-		)
-		(fill
-			(color 0 0 0 0)
-		)
-		(property "Sheetname" "left"
-			(at 22.86 24.6884 0)
-			(show_name no)
-			(do_not_autoplace no)
-			(effects
-				(font
-					(size 1.27 1.27)
-				)
-				(justify left bottom)
-			)
-		)
-		(property "Sheetfile" "keyboard.kicad_sch"
-			(at 22.86 93.2946 0)
-			(show_name no)
-			(do_not_autoplace no)
-			(effects
-				(font
-					(size 1.27 1.27)
-				)
-				(justify left top)
-			)
-		)
-		(instances
-			(project "split keyboard"
-				(path "/e1af24d2-b379-41bc-99d4-76686fb1dd1a"
-					(page "2")
-				)
-			)
